Commit message: diff_drive_controller works. Try to add imu_broadcaster without success

File: curt_mini/models/curt_mini/gazebo.xacro (robot description, xacro)
@@ -24,7 +24,9 @@
   <!-- IMU -->
   <gazebo reference="imu_link">
-    <sensor name="br_imu" type="imu">
+    <sensor name="imu_sensor" type="imu">
       <always_on>true</always_on>
       <update_rate>100</update_rate>
+      <visualize>true</visualize>
+      <!-- <topic>imu</topic> -->
       <imu>
         <angular_velocity>
@@ -69,11 +71,4 @@
         </linear_acceleration>
       </imu>
-      <plugin name="bytes_imu" filename="libgazebo_ros_imu_sensor.so">
-        <ros>
-          <namespace>imu</namespace>
-          <remapping>~/out:=data</remapping>
-        </ros>
-        <initial_orientation_as_reference>false</initial_orientation_as_reference>
-      </plugin>
     </sensor>
   </gazebo>

File: curt_mini/models/curt_mini/ros2_control.xacro (robot description, xacro)
@@ -42,3 +42,22 @@
     </joint>
   </ros2_control>
+  <xacro:if value="$(arg simulation)">
+    <ros2_control name="Sensors" type="system">
+      <hardware>
+        <plugin>gz_ros2_control/GazeboSystem</plugin>
+      </hardware>
+      <sensor name="imu_sensor">
+        <state_interface name="orientation.x"/>
+        <state_interface name="orientation.y"/>
+        <state_interface name="orientation.z"/>
+        <state_interface name="orientation.w"/>
+        <state_interface name="angular_velocity.x"/>
+        <state_interface name="angular_velocity.y"/>
+        <state_interface name="angular_velocity.z"/>
+        <state_interface name="linear_acceleration.x"/>
+        <state_interface name="linear_acceleration.y"/>
+        <state_interface name="linear_acceleration.z"/>
+      </sensor>
+    </ros2_control>
+  </xacro:if>
 </robot>

File: curt_mini/models/curt_mini/sensors.xacro (robot description, xacro)
@@ -9,4 +9,11 @@
     <origin xyz="0.062 0.0 0.015" rpy="0.0 0.0 ${pi/2}"/>
   </joint>
-  <link name="imu_link" />
+  <link name="imu_link">
+    <inertial>
+      <mass value="0.01"/>
+      <inertia ixx="1e-6" ixy="0" ixz="0"
+               iyy="1e-6" iyz="0"
+               izz="1e-6"/>
+    </inertial>
+  </link>
 </robot>

Commit message: :tada: imu is well simualed in gazebo
- add the sensors plugin in the world.sdf file
- remove the IMU Broadcaster controller, we use the gazebo plugin
- the gazebo reference uses the link name of the imu !

File: curt_mini/models/curt_mini/gazebo.xacro (robot description, xacro)
@@ -25,51 +25,52 @@
   <gazebo reference="imu_link">
     <sensor name="imu_sensor" type="imu">
-      <always_on>true</always_on>
-      <update_rate>100</update_rate>
-      <visualize>true</visualize>
-      <!-- <topic>imu</topic> -->
-      <imu>
-        <angular_velocity>
-          <x>
-            <noise type="gaussian">
-              <mean>0.0</mean>
-              <stddev>2e-4</stddev>
-            </noise>
-          </x>
-          <y>
-            <noise type="gaussian">
-              <mean>0.0</mean>
-              <stddev>2e-4</stddev>
-            </noise>
-          </y>
-          <z>
-            <noise type="gaussian">
-              <mean>0.0</mean>
-              <stddev>2e-4</stddev>
-            </noise>
-          </z>
-        </angular_velocity>
-        <linear_acceleration>
-          <x>
-            <noise type="gaussian">
-              <mean>0.0</mean>
-              <stddev>1.7e-2</stddev>
-            </noise>
-          </x>
-          <y>
-            <noise type="gaussian">
-              <mean>0.0</mean>
-              <stddev>1.7e-2</stddev>
-            </noise>
-          </y>
-          <z>
-            <noise type="gaussian">
-              <mean>0.0</mean>
-              <stddev>1.7e-2</stddev>
-            </noise>
-          </z>
-        </linear_acceleration>
-      </imu>
+        <always_on>true</always_on>
+        <update_rate>50</update_rate>
+        <visualize>true</visualize>
+        <topic>imu</topic>
+        <imu>
+          <angular_velocity>
+            <x>
+              <noise type="gaussian">
+                <mean>0.0</mean>
+                <stddev>2e-4</stddev>
+              </noise>
+            </x>
+            <y>
+              <noise type="gaussian">
+                <mean>0.0</mean>
+                <stddev>2e-4</stddev>
+              </noise>
+            </y>
+            <z>
+              <noise type="gaussian">
+                <mean>0.0</mean>
+                <stddev>2e-4</stddev>
+              </noise>
+            </z>
+          </angular_velocity>
+          <linear_acceleration>
+            <x>
+              <noise type="gaussian">
+                <mean>0.0</mean>
+                <stddev>1.7e-2</stddev>
+              </noise>
+            </x>
+            <y>
+              <noise type="gaussian">
+                <mean>0.0</mean>
+                <stddev>1.7e-2</stddev>
+              </noise>
+            </y>
+            <z>
+              <noise type="gaussian">
+                <mean>0.0</mean>
+                <stddev>1.7e-2</stddev>
+              </noise>
+            </z>
+          </linear_acceleration>
+        </imu>
     </sensor>
+    <material>Gazebo/Grey</material>
   </gazebo>
   <gazebo>

File: curt_mini/models/curt_mini/ros2_control.xacro (robot description, xacro)
@@ -42,22 +42,3 @@
     </joint>
   </ros2_control>
-  <xacro:if value="$(arg simulation)">
-    <ros2_control name="Sensors" type="system">
-      <hardware>
-        <plugin>gz_ros2_control/GazeboSystem</plugin>
-      </hardware>
-      <sensor name="imu_sensor">
-        <state_interface name="orientation.x"/>
-        <state_interface name="orientation.y"/>
-        <state_interface name="orientation.z"/>
-        <state_interface name="orientation.w"/>
-        <state_interface name="angular_velocity.x"/>
-        <state_interface name="angular_velocity.y"/>
-        <state_interface name="angular_velocity.z"/>
-        <state_interface name="linear_acceleration.x"/>
-        <state_interface name="linear_acceleration.y"/>
-        <state_interface name="linear_acceleration.z"/>
-      </sensor>
-    </ros2_control>
-  </xacro:if>
 </robot>

Commit message: modify prefix because the robot is dissociated, does not move in rviz

File: curt_mini/models/curt_mini/gazebo.xacro (robot description, xacro)
@@ -3,25 +3,25 @@
   <!-- Some properties -->
   <xacro:include filename="$(find curt_mini)/models/curt_mini/properties.xacro" />
-  <gazebo reference="base_link">
+  <gazebo reference="$(arg prefix)base_link">
     <material>Gazebo/Grey</material>
   </gazebo>
-  <gazebo reference="front_left_wheel">
+  <gazebo reference="$(arg prefix)front_left_wheel">
     <xacro:wheel_ode_params />
     <material>Gazebo/Black</material>
   </gazebo>
-  <gazebo reference="front_right_wheel">
+  <gazebo reference="$(arg prefix)front_right_wheel">
     <xacro:wheel_ode_params />
     <material>Gazebo/Black</material>
   </gazebo>
-  <gazebo reference="back_left_wheel">
+  <gazebo reference="$(arg prefix)back_left_wheel">
     <xacro:wheel_ode_params />
     <material>Gazebo/Black</material>
   </gazebo>
-  <gazebo reference="back_right_wheel">
+  <gazebo reference="$(arg prefix)back_right_wheel">
     <xacro:wheel_ode_params />
     <material>Gazebo/Black</material>
   </gazebo>
   <!-- IMU -->
-  <gazebo reference="imu_link">
+  <gazebo reference="$(arg prefix)imu_link">
     <sensor name="imu_sensor" type="imu">
         <always_on>true</always_on>
@@ -74,4 +74,35 @@
     <material>Gazebo/Grey</material>
   </gazebo>
+  <!-- LIDAR -->
+  <gazebo reference="$(arg prefix)lidar_link">
+    <sensor name='gpu_lidar' type='gpu_lidar'>"
+        <pose relative_to='$(arg prefix)lidar_link'>0 0 0 0 0 0</pose>
+        <topic>lidar</topic>
+        <update_rate>1</update_rate>
+        <ray>
+            <scan>
+                <horizontal>
+                    <samples>640</samples>
+                    <resolution>1</resolution>
+                    <min_angle>-1.396263</min_angle>
+                    <max_angle>1.396263</max_angle>
+                </horizontal>
+                <vertical>
+                    <samples>1</samples>
+                    <resolution>0.01</resolution>
+                    <min_angle>0</min_angle>
+                    <max_angle>0</max_angle>
+                </vertical>
+            </scan>
+            <range>
+                <min>0.08</min>
+                <max>10.0</max>
+                <resolution>0.01</resolution>
+            </range>
+        </ray>
+        <always_on>1</always_on>
+        <visualize>true</visualize>
+    </sensor>
+  </gazebo>
   <gazebo>
     <plugin filename="gz-sim-pose-publisher-system" name="gz::sim::systems::PosePublisher">

File: curt_mini/models/curt_mini/robot.urdf.xacro (robot description, xacro)
@@ -6,4 +6,5 @@
   <xacro:arg name="gazebo_controllers" default="$(arg path)/config/ros2_control_simulation.yaml" />
   <xacro:arg name="simulation" default="False" />
+  <xacro:arg name="prefix" default="curt_mini/"/>
   <!-- Import ros2_control -->
   <xacro:include filename="$(find curt_mini)/models/curt_mini/ros2_control.xacro" />
@@ -12,8 +13,8 @@
   <!-- Include sensors -->
   <xacro:include filename="$(find curt_mini)/models/curt_mini/sensors.xacro" />
-  <link name="base_link" />
+  <link name="$(arg prefix)base_link" />
   <!-- Chassis link at same position as base_link, as root is not allowed to have inertial
   information -->
-  <link name="chassis">
+  <link name="$(arg prefix)chassis">
     <inertial>
       <origin xyz="0.011876 0.003999 0.048645" rpy="0 0 0" />
@@ -39,8 +40,8 @@
   </link>
   <joint name="base_to_chassis" type="fixed">
-    <parent link="base_link" />
-    <child link="chassis" />
+    <parent link="$(arg prefix)base_link" />
+    <child link="$(arg prefix)chassis" />
   </joint>
-  <link name="front_right_wheel">
+  <link name="$(arg prefix)front_right_wheel">
     <inertial>
       <origin xyz="-2.8086E-05 0.013016 2.8089E-05" rpy="0 0 0" />
@@ -67,11 +68,11 @@
   <joint name="front_right_motor" type="continuous">
     <origin xyz="0.25995 -0.258 -0.030204" rpy="0 0 0" />
-    <parent link="base_link" />
-    <child link="front_right_wheel" />
+    <parent link="$(arg prefix)base_link" />
+    <child link="$(arg prefix)front_right_wheel" />
     <axis xyz="0 1 0" />
     <dynamics damping="1.0" />
     <limit effort="${max_effort}" velocity="${max_wheel_velocity}" />
   </joint>
-  <link name="front_left_wheel">
+  <link name="$(arg prefix)front_left_wheel">
     <inertial>
       <origin xyz="2.8086E-05 -0.013016 2.8089E-05" rpy="0 0 0" />
@@ -98,11 +99,11 @@
   <joint name="front_left_motor" type="continuous">
     <origin xyz="0.25995 0.258 -0.030204" rpy="0 0 0" />
-    <parent link="base_link" />
-    <child link="front_left_wheel" />
+    <parent link="$(arg prefix)base_link" />
+    <child link="$(arg prefix)front_left_wheel" />
     <axis xyz="0 1 0" />
     <dynamics damping="1.0" />
     <limit effort="${max_effort}" velocity="${max_wheel_velocity}" />
   </joint>
-  <link name="back_right_wheel">
+  <link name="$(arg prefix)back_right_wheel">
     <inertial>
       <origin xyz="-2.8086E-05 0.013016 2.8089E-05" rpy="0 0 0" />
@@ -129,11 +130,11 @@
   <joint name="back_right_motor" type="continuous">
     <origin xyz="-0.26 -0.258 -0.022755" rpy="0 0 0" />
-    <parent link="base_link" />
-    <child link="back_right_wheel" />
+    <parent link="$(arg prefix)base_link" />
+    <child link="$(arg prefix)back_right_wheel" />
     <axis xyz="0 1 0" />
     <dynamics damping="1.0" />
     <limit effort="${max_effort}" velocity="${max_wheel_velocity}" />
   </joint>
-  <link name="back_left_wheel">
+  <link name="$(arg prefix)back_left_wheel">
     <inertial>
       <origin xyz="2.8086E-05 -0.013016 2.8089E-05" rpy="0 0 0" />
@@ -160,6 +161,6 @@
   <joint name="back_left_motor" type="continuous">
     <origin xyz="-0.26 0.258 -0.022755" rpy="0 0 0" />
-    <parent link="base_link" />
-    <child link="back_left_wheel" />
+    <parent link="$(arg prefix)base_link" />
+    <child link="$(arg prefix)back_left_wheel" />
     <axis xyz="0 1 0" />
     <dynamics damping="1.0" />

File: curt_mini/models/curt_mini/sensors.xacro (robot description, xacro)
@@ -5,9 +5,9 @@
   <!-- LPResearch CANAL3 IMU -->
   <joint name="base_link_to_imu" type="fixed">
-    <parent link="base_link" />
-    <child link="imu_link" />
+    <parent link="$(arg prefix)base_link" />
+    <child link="$(arg prefix)imu_link" />
     <origin xyz="0.062 0.0 0.015" rpy="0.0 0.0 ${pi/2}"/>
   </joint>
-  <link name="imu_link">
+  <link name="$(arg prefix)imu_link">
     <inertial>
       <mass value="0.01"/>
@@ -17,3 +17,10 @@
     </inertial>
   </link>
+  <!-- Lidar UTM-30LX-EW -->
+  <joint name="base_link_to_lidar" type="fixed">
+    <parent link="$(arg prefix)base_link" />
+    <child link="$(arg prefix)lidar_link" />
+    <origin xyz="-0.162 0.0 0.315" rpy="${pi/2} 0.0 ${pi/2}"/>
+  </joint>
+  <link name="$(arg prefix)lidar_link"/>
 </robot>

Commit message: lidar works but odom does not publish anymore

File: curt_mini/models/curt_mini/gazebo.xacro (robot description, xacro)
@@ -76,6 +76,8 @@
   <!-- LIDAR -->
   <gazebo reference="$(arg prefix)lidar_link">
-    <sensor name='gpu_lidar' type='gpu_lidar'>"
-        <pose relative_to='$(arg prefix)lidar_link'>0 0 0 0 0 0</pose>
+    <sensor name='lidar' type='gpu_lidar'>"
+        <pose relative_to='lidar_link'>0 0 0 0 0 0</pose>
+        <!-- <frame_id>lidar_link</frame_id> -->
+        <gz_frame_id>lidar_link</gz_frame_id>
         <topic>lidar</topic>
         <update_rate>1</update_rate>

File: curt_mini/models/curt_mini/robot.urdf.xacro (robot description, xacro)
@@ -6,5 +6,5 @@
   <xacro:arg name="gazebo_controllers" default="$(arg path)/config/ros2_control_simulation.yaml" />
   <xacro:arg name="simulation" default="False" />
-  <xacro:arg name="prefix" default="curt_mini/"/>
+  <xacro:arg name="prefix" default=""/>
   <!-- Import ros2_control -->
   <xacro:include filename="$(find curt_mini)/models/curt_mini/ros2_control.xacro" />

File: curt_mini/models/curt_mini/sensors.xacro (robot description, xacro)
@@ -21,6 +21,20 @@
     <parent link="$(arg prefix)base_link" />
     <child link="$(arg prefix)lidar_link" />
-    <origin xyz="-0.162 0.0 0.315" rpy="${pi/2} 0.0 ${pi/2}"/>
+    <origin xyz="0.162 0.0 0.315" rpy="0.0 0.0 -${pi/2}"/>
   </joint>
-  <link name="$(arg prefix)lidar_link"/>
+  <!-- add collision for gazebo not to ignore the link-->
+  <link name="$(arg prefix)lidar_link">
+    <collision name="lidar_collision">
+    <origin xyz="0 0 0" rpy="0 0 0"/>
+    <geometry>
+      <box size="0.01 0.01 0.01"/>
+    </geometry>
+    </collision>
+    <inertial>
+      <mass value="0.01"/>
+      <inertia ixx="1e-6" ixy="0" ixz="0"
+               iyy="1e-6" iyz="0"
+               izz="1e-6"/>
+    </inertial>
+  </link>
 </robot>
